File: MMDVM_Hat.sch (KiCad schematic (older format))
At the start: 66 parts, among them J1 Radio, J2 Raspberry_Pi_2_3, J3 Serial Display, J4 FP_LEDs, J5 Radio, J6 STLink, J7 GS2, Q1 IRLML2060, Q2 2N7002, U1 LD1117S33TR, U2 STM32F722RETx, X1 TCXO, Y1 8 MHz

Commit message: Revision 0.1
Parts:
- removed J4: FP_LEDs, Pin_Headers:Pin_Header_Straight_2x05_Pitch2.54mm, symbol conn:Conn_02x05_Top_Bottom
- added D10: POCSAG, LEDs:LED_0603, symbol device:LED_Small
- added J4: Panel LEDs, Pin_Headers:Pin_Header_Straight_2x10_Pitch2.00mm, symbol conn:Conn_02x10_Odd_Even
- added R33: 1k5, Resistors_SMD:R_0603, symbol device:R_Small
Connections:
- net labels added: POCSAG_LED
- wire segments 276 -> 336
- no-connect marks 57 -> 55
Other:
- moved on the sheet: U1, U2

Commit message: Add value for R19 and BOM
Parts:
- C1, C5: symbol device:CP_Small -> MMDVM_Hat-rescue:CP_Small-device; MFR (none) -> AVX; MPN (none) -> THJA106K006AJN; SPN (none) -> 581-THJA106K006AJN; SPR (none) -> Mouser; SPURL (none) -> -
- C10, C12, C13, C16, C2, C21, C22, C24, C3: symbol device:C_Small -> MMDVM_Hat-rescue:C_Small-device; MFR (none) -> KEMET; MPN (none) -> C0603T104K3RALTU; SPN (none) -> 80-C0603T104K3RALTU; SPR (none) -> Mouser; SPURL (none) -> -
- C11, C19, C20, C23, C25: symbol device:C_Small -> MMDVM_Hat-rescue:C_Small-device; MFR (none) -> Murata Electronics; MPN (none) -> GRM188R61C475KAAJD; SPN (none) -> 81-GRM188R61C475KAJD; SPR (none) -> Mouser; SPURL (none) -> -
- C14, C15: symbol device:C_Small -> MMDVM_Hat-rescue:C_Small-device; MFR (none) -> KEMET; MPN (none) -> C0603C471K4RACTU; SPN (none) -> 80-C0603C471K4R; SPR (none) -> Mouser; SPURL (none) -> -
- C17, C18: symbol device:C_Small -> MMDVM_Hat-rescue:C_Small-device; MFR (none) -> KEMET; MPN (none) -> C0603C200K4GACTU; SPN (none) -> 80-C0603C200K4G; SPR (none) -> Mouser; SPURL (none) -> -
- C7: symbol device:C_Small -> MMDVM_Hat-rescue:C_Small-device; MFR (none) -> KEMET; MPN (none) -> C0603C106M7PACTU; SPN (none) -> 80-C0603C106M7P; SPR (none) -> Mouser; SPURL (none) -> -
- D1, D9: symbol device:LED_Small -> MMDVM_Hat-rescue:LED_Small-device; MFR (none) -> Kingbright; MPN (none) -> APT1608SGC; SPN (none) -> 604-APT1608SGC; SPR (none) -> Mouser; SPURL (none) -> -
- D10, D5: symbol device:LED_Small -> MMDVM_Hat-rescue:LED_Small-device; MFR (none) -> Kingbright; MPN (none) -> APT1608VBC/D; SPN (none) -> 604-APT1608VBC/D; SPR (none) -> Mouser; SPURL (none) -> -
- D2, D4, D6: symbol device:LED_Small -> MMDVM_Hat-rescue:LED_Small-device; MFR (none) -> Kingbright; MPN (none) -> APT1608SURCK; SPN (none) -> 604-APT1608SURCK; SPR (none) -> Mouser; SPURL (none) -> -
- D3, D8: symbol device:LED_Small -> MMDVM_Hat-rescue:LED_Small-device; MFR (none) -> Kingbright; MPN (none) -> APT1608SYC; SPN (none) -> 604-APT1608SYC; SPR (none) -> Mouser; SPURL (none) -> -
- D7: symbol device:LED_Small -> MMDVM_Hat-rescue:LED_Small-device; MFR (none) -> Kingbright; MPN (none) -> APT1608SECK; SPN (none) -> 604-APT1608SECK; SPR (none) -> Mouser; SPURL (none) -> -
- J1: symbol conn:DB9_Female_MountingHoles -> MMDVM_Hat-rescue:DB9_Female_MountingHoles-conn; MFR (none) -> TE Connectivity / AMP; MPN (none) -> 1734354-1; SPN (none) -> 571-1734354-1; SPR (none) -> Mouser; SPURL (none) -> -
- J2: symbol conn:Raspberry_Pi_2_3 -> MMDVM_Hat-rescue:Raspberry_Pi_2_3-conn; MFR (none) -> Harwin; MPN (none) -> M20-7832046; SPN (none) -> 855-M20-7832046; SPR (none) -> Mouser; SPURL (none) -> -
- J3, J6: symbol conn:Conn_01x04 -> MMDVM_Hat-rescue:Conn_01x04-conn; MFR (none) -> Wurth Electronics; MPN (none) -> 61300411121; SPN (none) -> 710-61300411121; SPR (none) -> Mouser; SPURL (none) -> -
- J4: symbol conn:Conn_02x10_Odd_Even -> MMDVM_Hat-rescue:Conn_02x10_Odd_Even-conn; MFR (none) -> 3M Electronic Solutions Division; MPN (none) -> 951210-8622-AR; SPN (none) -> 517-951210-8622-AR; SPR (none) -> Mouser; SPURL (none) -> -
- J5: symbol conn:Conn_01x07 -> MMDVM_Hat-rescue:Conn_01x07-conn; MFR (none) -> Wurth Electronics; MPN (none) -> 61300711121; SPN (none) -> 710-61300711121; SPR (none) -> Mouser; SPURL (none) -> -
- J7: symbol conn:GS2 -> MMDVM_Hat-rescue:GS2-conn; SPURL (none) -> -
- L1: symbol device:L_Core_Ferrite_Small -> MMDVM_Hat-rescue:L_Core_Ferrite_Small-device; MFR (none) -> Murata Electronics; MPN (none) -> LQM18FN100M00D; SPN (none) -> 81-LQM18FN100M00D; SPR (none) -> Mouser; SPURL (none) -> -
- L2: symbol device:Ferrite_Bead_Small -> MMDVM_Hat-rescue:Ferrite_Bead_Small-device; MFR (none) -> Wurth Electronics; MPN (none) -> 742863160; SPN (none) -> 710-742863160; SPR (none) -> Mouser; SPURL (none) -> -
- Q1: symbol device:Q_NMOS_GSD -> MMDVM_Hat-rescue:Q_NMOS_GSD-device; MFR (none) -> Infineon Technologies; MPN (none) -> IRLML2060TRPBF; SPN (none) -> 942-IRLML2060TRPBF; SPR (none) -> Mouser; SPURL (none) -> -
- Q2: symbol device:Q_NMOS_GSD -> MMDVM_Hat-rescue:Q_NMOS_GSD-device; MFR (none) -> ON Semiconductor / Fairchild; MPN (none) -> 2N7002; SPN (none) -> 512-2N7002; SPR (none) -> Mouser; SPURL (none) -> -
- R1, R11, R2, R33, R4, R5, R6, R7, R8, R9: symbol device:R_Small -> MMDVM_Hat-rescue:R_Small-device; MFR (none) -> Panasonic; MPN (none) -> ERJ-3EKF1501V; SPN (none) -> 667-ERJ-3EKF1501V; SPR (none) -> Mouser; SPURL (none) -> -
- R10, R3: symbol device:R_Small -> MMDVM_Hat-rescue:R_Small-device; MFR (none) -> Panasonic; MPN (none) -> ERJ-PB3B1002V; SPN (none) -> 667-ERJ-PB3B1002V; SPR (none) -> Mouser; SPURL (none) -> -
- R12, R16, R18: symbol device:R_Small -> MMDVM_Hat-rescue:R_Small-device; MFR (none) -> Panasonic; MPN (none) -> ERJ-3EKF4702V; SPN (none) -> 667-ERJ-3EKF4702V; SPR (none) -> Mouser; SPURL (none) -> -
- R13, R14: symbol device:R_Small -> MMDVM_Hat-rescue:R_Small-device; MFR (none) -> Panasonic; MPN (none) -> ERJ-U03F3300V; SPN (none) -> 667-ERJ-U03F3300V; SPR (none) -> Mouser; SPURL (none) -> -
- R15: symbol device:R_Small -> MMDVM_Hat-rescue:R_Small-device; MFR (none) -> Panasonic; MPN (none) -> ERJ-3EKF1004V; SPN (none) -> 667-ERJ-3EKF1004V; SPR (none) -> Mouser; SPURL (none) -> -
- R17: symbol device:R_Small -> MMDVM_Hat-rescue:R_Small-device; MFR (none) -> Panasonic; MPN (none) -> ERJ-3EKF4701V; SPN (none) -> 667-ERJ-3EKF4701V; SPR (none) -> Mouser; SPURL (none) -> -
- R19: value R -> 1M; symbol device:R -> MMDVM_Hat-rescue:R-device; MFR (none) -> Panasonic; MPN (none) -> ERJ-3EKF1004V; SPN (none) -> 667-ERJ-3EKF1004V; SPR (none) -> Mouser; SPURL (none) -> -
- RV1: symbol device:POT -> MMDVM_Hat-rescue:POT-device; MFR (none) -> Bourns; MPN (none) -> 3296Y-1-104LF; SPN (none) -> 652-3296Y-1-104LF; SPR (none) -> Mouser; SPURL (none) -> -
- TP1: symbol device:TEST -> MMDVM_Hat-rescue:TEST-device; SPURL (none) -> -
- U1: symbol regul:LD1117S33TR_SOT223 -> MMDVM_Hat-rescue:LD1117S33TR_SOT223-regul; MFR (none) -> STMicroelectronics; MPN (none) -> LD1117S33TR; SPN (none) -> 511-LD1117S33; SPR (none) -> Mouser; SPURL (none) -> -
- U2: symbol MCU_ST_STM32F7:STM32F722RETx -> MMDVM_Hat-rescue:STM32F722RETx-MCU_ST_STM32F7; MFR (none) -> STMicroelectronics; MPN (none) -> STM32F722RET6; SPN (none) -> 511-STM32F722RET6; SPR (none) -> Mouser; SPURL (none) -> -
- X1: symbol Oscillators:ASV-xxxMHz -> MMDVM_Hat-rescue:ASV-xxxMHz-Oscillators; MFR (none) -> Fox; MPN (none) -> FOX924B-12; SPN (none) -> 559-FOX924B-12; SPR (none) -> Mouser; SPURL (none) -> -
- Y1: symbol device:Crystal_Small -> MMDVM_Hat-rescue:Crystal_Small-device; MFR (none) -> ABRACON; MPN (none) -> ABM3-8.000MHz-D2Y-T; SPN (none) -> 815-ABM3-8-D2Y-T; SPR (none) -> Mouser; SPURL (none) -> -

Commit message: Change Case code for 47u caps
Parts:
- C1, C5: MPN THJA106K006AJN -> F931C106KAA; SPN 581-THJA106K006AJN -> 647-F931C106KAA
Changed lines of the file:
@@
 F 1 "10u" H 838 955 50 0000 L CNN
 F 2 "Capacitors_Tantalum_SMD:CP_Tantalum_Case-A_EIA-3216-18_Reflow" H 750 1000 50 0001 C CNN
-F 3 "https://www.mouser.de/datasheet/2/40/thj-776995.pdf" H 750 1000 50 0001 C CNN
+F 3 "https://www.mouser.de/datasheet/2/40/f93-776559.pdf" H 750 1000 50 0001 C CNN
 F 4 "AVX" H 0 0 50 0001 C CNN "MFR"
-F 5 "THJA106K006AJN" H 0 0 50 0001 C CNN "MPN"
+F 5 "F931C106KAA" H 0 0 50 0001 C CNN "MPN"
 F 6 "Mouser" H 0 0 50 0001 C CNN "SPR"
-F 7 "581-THJA106K006AJN" H 0 0 50 0001 C CNN "SPN"
+F 7 "647-F931C106KAA" H 0 0 50 0001 C CNN "SPN"
 F 8 "-" H 0 0 50 0001 C CNN "SPURL"
 	1    750  1000
@@
 F 1 "10u" H 2388 955 50 0000 L CNN
 F 2 "Capacitors_Tantalum_SMD:CP_Tantalum_Case-A_EIA-3216-18_Reflow" H 2300 1000 50 0001 C CNN
-F 3 "https://www.mouser.de/datasheet/2/40/thj-776995.pdf" H 2300 1000 50 0001 C CNN
+F 3 "https://www.mouser.de/datasheet/2/40/f93-776559.pdf" H 2300 1000 50 0001 C CNN
 F 4 "AVX" H 0 0 50 0001 C CNN "MFR"
-F 5 "THJA106K006AJN" H 0 0 50 0001 C CNN "MPN"
+F 5 "F931C106KAA" H 0 0 50 0001 C CNN "MPN"
 F 6 "Mouser" H 0 0 50 0001 C CNN "SPR"
-F 7 "581-THJA106K006AJN" H 0 0 50 0001 C CNN "SPN"
+F 7 "647-F931C106KAA" H 0 0 50 0001 C CNN "SPN"
 F 8 "-" H 0 0 50 0001 C CNN "SPURL"
 	1    2300 1000

Commit message: Re-add lost C4
Parts:
- added C4: 100n, Capacitors_SMD:C_0603, symbol MMDVM_Hat-rescue:C_Small-device
Connections:
- wire segments 336 -> 341
Changed lines of the file:
@@
 Sheet 1 2
 Title "MMDVM-F7-Hat"
-Date "2018-06-29"
+Date "2018-07-23"
 Rev "0.1"
 Comp "DB9MAT, DF2ET"
@@
 P 9750 2150
 F 0 "#PWR013" H 9750 2000 50 0001 C CNN
-F 1 "+3V3" V 9650 2150 50 0000 C CNN
+F 1 "+3V3" H 9700 2300 50 0000 C CNN
 F 2 "" H 9750 2150 50 0001 C CNN
 F 3 "" H 9750 2150 50 0001 C CNN
@@
 L MMDVM_Hat-rescue:C_Small-device C21
 U 1 1 5B24A2E2
-P 9400 1750
-F 0 "C21" V 9600 1750 50 0000 C CNN
-F 1 "100n" V 9500 1750 50 0000 C CNN
-F 2 "Capacitors_SMD:C_0603" H 9400 1750 50 0001 C CNN
-F 3 "https://www.mouser.de/datasheet/2/212/KEM_C1027_X7R_COTS_SMD-1099449.pdf" H 9400 1750 50 0001 C CNN
-F 4 "KEMET" H 0 0 50 0001 C CNN "MFR"
-F 5 "C0603T104K3RALTU" H 0 0 50 0001 C CNN "MPN"
-F 6 "Mouser" H 0 0 50 0001 C CNN "SPR"
-F 7 "80-C0603T104K3RALTU" H 0 0 50 0001 C CNN "SPN"
-F 8 "-" H 0 0 50 0001 C CNN "SPURL"
-	1    9400 1750
+P 9000 1850
+F 0 "C21" V 9200 1850 50 0000 C CNN
+F 1 "100n" V 9100 1850 50 0000 C CNN
+F 2 "Capacitors_SMD:C_0603" H 9000 1850 50 0001 C CNN
+F 3 "https://www.mouser.de/datasheet/2/212/KEM_C1027_X7R_COTS_SMD-1099449.pdf" H 9000 1850 50 0001 C CNN
+F 4 "KEMET" H -400 100 50 0001 C CNN "MFR"
+F 5 "C0603T104K3RALTU" H -400 100 50 0001 C CNN "MPN"
+F 6 "Mouser" H -400 100 50 0001 C CNN "SPR"
+F 7 "80-C0603T104K3RALTU" H -400 100 50 0001 C CNN "SPN"
+F 8 "-" H -400 100 50 0001 C CNN "SPURL"
+	1    9000 1850
 	0    1    1    0
 $EndComp
@@
 L MMDVM_Hat-rescue:C_Small-device C20
 U 1 1 5B24F686
-P 9400 1600
-F 0 "C20" V 9171 1600 50 0000 C CNN
-F 1 "4u7" V 9262 1600 50 0000 C CNN
-F 2 "Capacitors_SMD:C_0603" H 9400 1600 50 0001 C CNN
-F 3 "https://www.mouser.de/datasheet/2/281/murata_03052018_GRM_Series_1-1310166.pdf" H 9400 1600 50 0001 C CNN
-F 4 "Murata Electronics" H 0 0 50 0001 C CNN "MFR"
-F 5 "GRM188R61C475KAAJD" H 0 0 50 0001 C CNN "MPN"
-F 6 "Mouser" H 0 0 50 0001 C CNN "SPR"
-F 7 "81-GRM188R61C475KAJD" H 0 0 50 0001 C CNN "SPN"
-F 8 "-" H 0 0 50 0001 C CNN "SPURL"
-	1    9400 1600
+P 9000 1700
+F 0 "C20" V 8771 1700 50 0000 C CNN
+F 1 "4u7" V 8862 1700 50 0000 C CNN
+F 2 "Capacitors_SMD:C_0603" H 9000 1700 50 0001 C CNN
+F 3 "https://www.mouser.de/datasheet/2/281/murata_03052018_GRM_Series_1-1310166.pdf" H 9000 1700 50 0001 C CNN
+F 4 "Murata Electronics" H -400 100 50 0001 C CNN "MFR"
+F 5 "GRM188R61C475KAAJD" H -400 100 50 0001 C CNN "MPN"
+F 6 "Mouser" H -400 100 50 0001 C CNN "SPR"
+F 7 "81-GRM188R61C475KAJD" H -400 100 50 0001 C CNN "SPN"
+F 8 "-" H -400 100 50 0001 C CNN "SPURL"
+	1    9000 1700
 	0    1    1    0
 $EndComp
@@
 L power:GND #PWR014
 U 1 1 5B25084E
-P 9200 1850
-F 0 "#PWR014" H 9200 1600 50 0001 C CNN
-F 1 "GND" H 9205 1677 50 0000 C CNN
-F 2 "" H 9200 1850 50 0001 C CNN
-F 3 "" H 9200 1850 50 0001 C CNN
-	1    9200 1850
+P 8800 1950
+F 0 "#PWR014" H 8800 1700 50 0001 C CNN
+F 1 "GND" H 8805 1777 50 0000 C CNN
+F 2 "" H 8800 1950 50 0001 C CNN
+F 3 "" H 8800 1950 50 0001 C CNN
+	1    8800 1950
 	1    0    0    -1
 $EndComp
@@
 	1    2250 3550
 	0    1    1    0
+$EndComp
+$Comp
+L MMDVM_Hat-rescue:C_Small-device C4
+U 1 1 5B5E0676
+P 9500 1950
+F 0 "C4" V 9700 1950 50 0000 C CNN
+F 1 "100n" V 9600 1950 50 0000 C CNN
+F 2 "Capacitors_SMD:C_0603" H 9500 1950 50 0001 C CNN
+F 3 "https://www.mouser.de/datasheet/2/212/KEM_C1027_X7R_COTS_SMD-1099449.pdf" H 9500 1950 50 0001 C CNN
+F 4 "KEMET" H -400 850 50 0001 C CNN "MFR"
+F 5 "C0603T104K3RALTU" H -400 850 50 0001 C CNN "MPN"
+F 6 "Mouser" H -400 850 50 0001 C CNN "SPR"
+F 7 "80-C0603T104K3RALTU" H -400 850 50 0001 C CNN "SPN"
+F 8 "-" H -400 850 50 0001 C CNN "SPURL"
+	1    9500 1950
+	-1   0    0    -1
+$EndComp
+$Comp
+L power:GND #PWR?
+U 1 1 5B5E094C
+P 9350 1600
+F 0 "#PWR?" H 9350 1350 50 0001 C CNN
+F 1 "GND" H 9355 1427 50 0000 C CNN
+F 2 "" H 9350 1600 50 0001 C CNN
+F 3 "" H 9350 1600 50 0001 C CNN
+	1    9350 1600
+	1    0    0    -1
 $EndComp
 Text GLabel 9050 2450 0    50   Input ~ 0
@@
 	9750 2150 9750 2250
 Wire Wire Line
-	9500 1750 9600 1750
-Wire Wire Line
-	9500 1600 9600 1600
-Wire Wire Line
-	9600 1600 9600 1750
-Wire Wire Line
-	9300 1750 9200 1750
-Wire Wire Line
-	9200 1750 9200 1850
-Wire Wire Line
-	9300 1600 9200 1600
-Wire Wire Line
-	9200 1600 9200 1750
-Wire Wire Line
-	9600 1300 9600 1600
+	9100 1850 9200 1850
+Wire Wire Line
+	9100 1700 9200 1700
+Wire Wire Line
+	9200 1700 9200 1850
+Wire Wire Line
+	8900 1850 8800 1850
+Wire Wire Line
+	8800 1850 8800 1950
+Wire Wire Line
+	8900 1700 8800 1700
+Wire Wire Line
+	8800 1700 8800 1850
+Wire Wire Line
+	9200 1400 9200 1700
 Wire Wire Line
 	10000 1250 10100 1250
@@
 Wire Wire Line
 	9600 800  9600 700
-Wire Wire Line
-	9250 2950 9150 2950
-Wire Wire Line
-	9150 2950 9150 2150
-Wire Wire Line
-	9150 2150 9600 2150
-Wire Wire Line
-	9600 1750 9600 2150
 Wire Wire Line
 	9250 2450 9050 2450
@@
 Wire Wire Line
 	3300 2400 3300 2450
+Wire Wire Line
+	9200 1400 9600 1400
+Wire Wire Line
+	9600 1400 9600 1300
+Wire Wire Line
+	9250 2950 9200 2950
+Wire Wire Line
+	9200 2950 9200 1850
+Wire Wire Line
+	9500 2150 9500 2050
+Wire Wire Line
+	9500 2150 9750 2150
+Wire Wire Line
+	9500 1850 9500 1550
+Wire Wire Line
+	9500 1550 9350 1550
+Wire Wire Line
+	9350 1550 9350 1600
 Connection ~ 1950 4650
 Connection ~ 2400 7450
@@
 Connection ~ 750  1200
 Connection ~ 750  800
-Connection ~ 9600 1750
-Connection ~ 9200 1750
-Connection ~ 9600 1600
+Connection ~ 8800 1850
+Connection ~ 9200 1700
 Connection ~ 10100 1250
 Connection ~ 9700 1100
@@
 Connection ~ 3000 2400
 Connection ~ 3300 2400
+Connection ~ 9200 1850
+Connection ~ 9750 2150
 NoConn ~ 9250 4350
 NoConn ~ 9250 4450

Commit message: Add Channel switch line (schematic only)
Parts:
- removed J5: Radio, Pin_Headers:Pin_Header_Straight_1x07_Pitch2.54mm, symbol MMDVM_Hat-rescue:Conn_01x07-conn
- added C6: 470p, Capacitors_SMD:C_0603, symbol MMDVM_Hat-rescue:C_Small-device
- added J5: Radio, symbol Connector_Generic:Conn_01x08
- added Q3: 2N7002, TO_SOT_Packages_SMD:SOT-23, symbol MMDVM_Hat-rescue:Q_NMOS_GSD-device
- added R34: 47k, Resistors_SMD:R_0603, symbol MMDVM_Hat-rescue:R_Small-device
- added R35: 330, Resistors_SMD:R_0603, symbol MMDVM_Hat-rescue:R_Small-device
Connections:
- net labels added: CH_SW, RADIO_CH_SW
- wire segments 341 -> 353
Other:
- note added: "Channel Switch Line"

Commit message: Use FET for channel switch
Parts:
- Q3: value 2N7002 -> IRLML2060
Changed lines of the file:
@@
 P 4900 3550
 F 0 "Q3" H 5105 3596 50  0000 L CNN
-F 1 "2N7002" H 5105 3505 50  0000 L CNN
+F 1 "IRLML2060" H 5105 3505 50  0000 L CNN
 F 2 "TO_SOT_Packages_SMD:SOT-23" H 5100 3650 50  0001 C CNN
 F 3 "https://www.mouser.de/datasheet/2/196/irlml2060pbf-1228502.pdf" H 4900 3550 50  0001 C CNN
