File: MMDVM_Hat.sch (KiCad schematic (older format))
At the start: 73 parts, among them J1 Radio, J2 Raspberry_Pi_2_3, J3 Serial Display, J4 Panel LEDs, J5 Radio, J6 STLink, J7 GS2, Q1 IRLML2060, Q2 2N7002, Q3 IRLML2060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

Commit message: Revision 0.2: Added FET for channel switching; Rename to MMDVM_RPT_Hat
Parts:
- C1, C5: symbol MMDVM_Hat-rescue:CP_Small-device -> MMDVM_Hat-rescue:CP_Small-device-MMDVM_Hat-rescue
- C10, C11, C12, C13, C14, C15, C16, C17, C18, C19, C2, C20, C21, C22, C23, C24, C25, C3, C4, C6, C7: symbol MMDVM_Hat-rescue:C_Small-device -> MMDVM_Hat-rescue:C_Small-device-MMDVM_Hat-rescue
- D1, D10, D2, D3, D4, D5, D6, D7, D8, D9: symbol MMDVM_Hat-rescue:LED_Small-device -> MMDVM_Hat-rescue:LED_Small-device-MMDVM_Hat-rescue
- J1: symbol MMDVM_Hat-rescue:DB9_Female_MountingHoles-conn -> MMDVM_Hat-rescue:DB9_Female_MountingHoles-conn-MMDVM_Hat-rescue
- J2: symbol MMDVM_Hat-rescue:Raspberry_Pi_2_3-conn -> MMDVM_Hat-rescue:Raspberry_Pi_2_3-conn-MMDVM_Hat-rescue
- J3, J6: symbol MMDVM_Hat-rescue:Conn_01x04-conn -> MMDVM_Hat-rescue:Conn_01x04-conn-MMDVM_Hat-rescue
- J4: symbol MMDVM_Hat-rescue:Conn_02x10_Odd_Even-conn -> MMDVM_Hat-rescue:Conn_02x10_Odd_Even-conn-MMDVM_Hat-rescue
- J5: footprint (none) -> Pin_Headers:Pin_Header_Straight_1x08_Pitch2.54mm; symbol Connector_Generic:Conn_01x08 -> MMDVM_Hat-rescue:Conn_01x08-Connector_Generic
- J7: symbol MMDVM_Hat-rescue:GS2-conn -> MMDVM_Hat-rescue:GS2-conn-MMDVM_Hat-rescue
- L1: symbol MMDVM_Hat-rescue:L_Core_Ferrite_Small-device -> MMDVM_Hat-rescue:L_Core_Ferrite_Small-device-MMDVM_Hat-rescue
- L2: symbol MMDVM_Hat-rescue:Ferrite_Bead_Small-device -> MMDVM_Hat-rescue:Ferrite_Bead_Small-device-MMDVM_Hat-rescue
- Q1, Q2, Q3: symbol MMDVM_Hat-rescue:Q_NMOS_GSD-device -> MMDVM_Hat-rescue:Q_NMOS_GSD-device-MMDVM_Hat-rescue
- R1, R10, R11, R12, R13, R14, R15, R16, R17, R18, R2, R3, R33, R34, R35, R4, R5, R6, R7, R8, R9: symbol MMDVM_Hat-rescue:R_Small-device -> MMDVM_Hat-rescue:R_Small-device-MMDVM_Hat-rescue
- R19: symbol MMDVM_Hat-rescue:R-device -> MMDVM_Hat-rescue:R-device-MMDVM_Hat-rescue
- RV1: symbol MMDVM_Hat-rescue:POT-device -> MMDVM_Hat-rescue:POT-device-MMDVM_Hat-rescue
- TP1: symbol MMDVM_Hat-rescue:TEST-device -> MMDVM_Hat-rescue:TEST-device-MMDVM_Hat-rescue
- U1: symbol MMDVM_Hat-rescue:LD1117S33TR_SOT223-regul -> MMDVM_Hat-rescue:LD1117S33TR_SOT223-regul-MMDVM_Hat-rescue
- U2: symbol MMDVM_Hat-rescue:STM32F722RETx-MCU_ST_STM32F7 -> MMDVM_Hat-rescue:STM32F722RETx-MCU_ST_STM32F7-MMDVM_Hat-rescue
- X1: symbol MMDVM_Hat-rescue:ASV-xxxMHz-Oscillators -> MMDVM_Hat-rescue:ASV-xxxMHz-Oscillators-MMDVM_Hat-rescue
- Y1: symbol MMDVM_Hat-rescue:Crystal_Small-device -> MMDVM_Hat-rescue:Crystal_Small-device-MMDVM_Hat-rescue
