File: Filter.sch (KiCad schematic (older format))
At the start: 36 parts, among them J8 GS3, U3 MCP6002, U4 MCP6002

Commit message: Add value for R19 and BOM
Parts:
- C26, C27, C31, C34, C36: symbol device:CP_Small -> MMDVM_Hat-rescue:CP_Small-device; MFR (none) -> AVX; MPN (none) -> F931A476KAA; SPN (none) -> 647-F931A476KAA; SPR (none) -> Mouser; SPURL (none) -> -
- C28, C32: symbol device:C_Small -> MMDVM_Hat-rescue:C_Small-device; MFR (none) -> KEMET; MPN (none) -> C0603C103K4RAC; SPN (none) -> 80-C0603C103K4RAC; SPR (none) -> Mouser; SPURL (none) -> -
- C29, C33: symbol device:C_Small -> MMDVM_Hat-rescue:C_Small-device; MFR (none) -> KEMET; MPN (none) -> C0603C393K4RACTU; SPN (none) -> 80-C0603C393K4R; SPR (none) -> Mouser; SPURL (none) -> -
- C30, C35: symbol device:C_Small -> MMDVM_Hat-rescue:C_Small-device; MFR (none) -> KEMET; MPN (none) -> C0603S102K4RACTU; SPN (none) -> 80-C0603S102K4R; SPR (none) -> Mouser; SPURL (none) -> -
- C37, C38: symbol device:C_Small -> MMDVM_Hat-rescue:C_Small-device; MFR (none) -> KEMET; MPN (none) -> C0603T104K3RALTU; SPN (none) -> 80-C0603T104K3RALTU; SPR (none) -> Mouser; SPURL (none) -> -
- J8: symbol conn:GS3 -> MMDVM_Hat-rescue:GS3-conn; SPURL (none) -> -
- R20: symbol device:R_Small -> MMDVM_Hat-rescue:R_Small-device; MFR (none) -> Panasonic; MPN (none) -> ERJ-PB3B1002V; SPN (none) -> 667-ERJ-PB3B1002V; SPR (none) -> Mouser; SPURL (none) -> -
- R21: symbol device:R_Small -> MMDVM_Hat-rescue:R_Small-device; MFR (none) -> Panasonic; MPN (none) -> ERJ-3EKF1001V; SPN (none) -> 667-ERJ-3EKF1001V; SPR (none) -> Mouser; SPURL (none) -> -
- R22: symbol device:R_Small -> MMDVM_Hat-rescue:R_Small-device; MFR (none) -> Panasonic; MPN (none) -> ERJ-3EKF2002V; SPN (none) -> 667-ERJ-3EKF2002V; SPR (none) -> Mouser; SPURL (none) -> -
- R23, R24, R25: symbol device:R_Small -> MMDVM_Hat-rescue:R_Small-device; MFR (none) -> Panasonic; MPN (none) -> ERJ-P03F2202V; SPN (none) -> 667-ERJ-P03F2202V; SPR (none) -> Mouser; SPURL (none) -> -
- R26, R30: symbol device:R_Small -> MMDVM_Hat-rescue:R_Small-device; MFR (none) -> Panasonic; MPN (none) -> ERJ-3EKF5101V; SPN (none) -> 667-ERJ-3EKF5101V; SPR (none) -> Mouser; SPURL (none) -> -
- R27, R28, R31, R32: symbol device:R_Small -> MMDVM_Hat-rescue:R_Small-device; MFR (none) -> Panasonic; MPN (none) -> ERJ-3EKF4701V; SPN (none) -> 667-ERJ-3EKF4701V; SPR (none) -> Mouser; SPURL (none) -> -
- R29: symbol device:R_Small -> MMDVM_Hat-rescue:R_Small-device; MFR (none) -> Panasonic; MPN (none) -> ERJ-3EKF3002V; SPN (none) -> 667-ERJ-3EKF3002V; SPR (none) -> Mouser; SPURL (none) -> -
- RV2: symbol device:POT -> MMDVM_Hat-rescue:POT-device; MFR (none) -> Bourns; MPN (none) -> 3314G-1-103E; SPN (none) -> 652-3314G-1-103E; SPR (none) -> Mouser; SPURL (none) -> -
- RV3: symbol device:POT -> MMDVM_Hat-rescue:POT-device; MFR (none) -> Bourns; MPN (none) -> 3214W-1-104E; SPN (none) -> 652-3214W-1-104E; SPR (none) -> Mouser; SPURL (none) -> -
- RV4: symbol device:POT -> MMDVM_Hat-rescue:POT-device; MFR (none) -> Bourns; MPN (none) -> 3214W-1-204E; SPN (none) -> 652-3214W-1-204E; SPR (none) -> Mouser; SPURL (none) -> -
- TP2, TP3, TP4, TP5: symbol device:TEST -> MMDVM_Hat-rescue:TEST-device; SPURL (none) -> -
- U3, U4: symbol linear:MCP6002-xMS -> MMDVM_Hat-rescue:MCP6002-xMS-linear; MFR (none) -> Microchip Technology; MPN (none) -> MCP6002-E/SN; SPN (none) -> 579-MCP6002-E/SN; SPR (none) -> Mouser; SPURL (none) -> -

Commit message: Correct part for 10nF capacitors
Parts:
- C28, C32: MPN C0603C103K4RAC -> C0603C103K2RECTU; SPN 80-C0603C103K4RAC -> 80-C0603C103K2REC
Changed lines of the file:
@@
 F 1 "10n" H 3842 2005 50 0000 L CNN
 F 2 "Capacitors_SMD:C_0603" H 3750 2050 50 0001 C CNN
-F 3 "https://www.mouser.de/datasheet/2/212/KEM_C1002_X7R_SMD-1102033.pdf" H 3750 2050 50 0001 C CNN
-F 4 "KEMET" H 0 0 50 0001 C CNN "MFR"
-F 5 "C0603C103K4RAC" H 0 0 50 0001 C CNN "MPN"
-F 6 "Mouser" H 0 0 50 0001 C CNN "SPR"
-F 7 "80-C0603C103K4RAC" H 0 0 50 0001 C CNN "SPN"
+F 3 "https://www.mouser.de/datasheet/2/212/KEM_C1090_X7R_ESD-1103328.pdf" H 3750 2050 50 0001 C CNN
+F 4 "KEMET" H 0 0 50 0001 C CNN "MFR"
+F 5 "C0603C103K2RECTU" H 0 0 50 0001 C CNN "MPN"
+F 6 "Mouser" H 0 0 50 0001 C CNN "SPR"
+F 7 "80-C0603C103K2REC" H 0 0 50 0001 C CNN "SPN"
 F 8 "-" H 0 0 50 0001 C CNN "SPURL"
 	1    3750 2050
@@
 F 1 "10n" H 2442 4155 50 0000 L CNN
 F 2 "Capacitors_SMD:C_0603" H 2350 4200 50 0001 C CNN
-F 3 "https://www.mouser.de/datasheet/2/212/KEM_C1002_X7R_SMD-1102033.pdf" H 2350 4200 50 0001 C CNN
-F 4 "KEMET" H 0 0 50 0001 C CNN "MFR"
-F 5 "C0603C103K4RAC" H 0 0 50 0001 C CNN "MPN"
-F 6 "Mouser" H 0 0 50 0001 C CNN "SPR"
-F 7 "80-C0603C103K4RAC" H 0 0 50 0001 C CNN "SPN"
+F 3 "https://www.mouser.de/datasheet/2/212/KEM_C1090_X7R_ESD-1103328.pdf" H 2350 4200 50 0001 C CNN
+F 4 "KEMET" H 0 0 50 0001 C CNN "MFR"
+F 5 "C0603C103K2RECTU" H 0 0 50 0001 C CNN "MPN"
+F 6 "Mouser" H 0 0 50 0001 C CNN "SPR"
+F 7 "80-C0603C103K2REC" H 0 0 50 0001 C CNN "SPN"
 F 8 "-" H 0 0 50 0001 C CNN "SPURL"
 	1    2350 4200

Commit message: Change Case code for 47u caps
Parts:
- C26, C27, C31, C34, C36: footprint Capacitors_Tantalum_SMD:CP_Tantalum_Case-A_EIA-3216-18_Reflow -> Capacitors_Tantalum_SMD:CP_EIA-6032-28_Kemet-C; MPN F931A476KAA -> TAJC476K016SNJ; SPN 647-F931A476KAA -> 581-TAJC476K016SNJ
Changed lines of the file:
@@
 F 0 "C26" V 1525 1750 50 0000 C CNN
 F 1 "47u" V 1616 1750 50 0000 C CNN
-F 2 "Capacitors_Tantalum_SMD:CP_Tantalum_Case-A_EIA-3216-18_Reflow" H 1750 1750 50 0001 C CNN
-F 3 "https://www.mouser.de/datasheet/2/40/f93-776559.pdf" H 1750 1750 50 0001 C CNN
+F 2 "Capacitors_Tantalum_SMD:CP_EIA-6032-28_Kemet-C" H 1750 1750 50 0001 C CNN
+F 3 "https://www.mouser.de/datasheet/2/40/taj-776811.pdf" H 1750 1750 50 0001 C CNN
 F 4 "AVX" H 0 0 50 0001 C CNN "MFR"
-F 5 "F931A476KAA" H 0 0 50 0001 C CNN "MPN"
-F 6 "Mouser" H 0 0 50 0001 C CNN "SPR"
-F 7 "647-F931A476KAA" H 0 0 50 0001 C CNN "SPN"
+F 5 "TAJC476K016SNJ" H 0 0 50 0001 C CNN "MPN"
+F 6 "Mouser" H 0 0 50 0001 C CNN "SPR"
+F 7 "581-TAJC476K016SNJ" H 0 0 50 0001 C CNN "SPN"
 F 8 "-" H 0 0 50 0001 C CNN "SPURL"
 	1    1750 1750
@@
 F 0 "C27" H 2162 1104 50 0000 R CNN
 F 1 "47u" H 2162 1195 50 0000 R CNN
-F 2 "Capacitors_Tantalum_SMD:CP_Tantalum_Case-A_EIA-3216-18_Reflow" H 2250 1150 50 0001 C CNN
-F 3 "https://www.mouser.de/datasheet/2/40/f93-776559.pdf" H 2250 1150 50 0001 C CNN
+F 2 "Capacitors_Tantalum_SMD:CP_EIA-6032-28_Kemet-C" H 2250 1150 50 0001 C CNN
+F 3 "https://www.mouser.de/datasheet/2/40/taj-776811.pdf" H 2250 1150 50 0001 C CNN
 F 4 "AVX" H 0 0 50 0001 C CNN "MFR"
-F 5 "F931A476KAA" H 0 0 50 0001 C CNN "MPN"
-F 6 "Mouser" H 0 0 50 0001 C CNN "SPR"
-F 7 "647-F931A476KAA" H 0 0 50 0001 C CNN "SPN"
+F 5 "TAJC476K016SNJ" H 0 0 50 0001 C CNN "MPN"
+F 6 "Mouser" H 0 0 50 0001 C CNN "SPR"
+F 7 "581-TAJC476K016SNJ" H 0 0 50 0001 C CNN "SPN"
 F 8 "-" H 0 0 50 0001 C CNN "SPURL"
 	1    2250 1150
@@
 F 0 "C31" H 3438 2896 50 0000 L CNN
 F 1 "47u" H 3438 2805 50 0000 L CNN
-F 2 "Capacitors_Tantalum_SMD:CP_Tantalum_Case-A_EIA-3216-18_Reflow" H 3350 2850 50 0001 C CNN
-F 3 "https://www.mouser.de/datasheet/2/40/f93-776559.pdf" H 3350 2850 50 0001 C CNN
+F 2 "Capacitors_Tantalum_SMD:CP_EIA-6032-28_Kemet-C" H 3350 2850 50 0001 C CNN
+F 3 "https://www.mouser.de/datasheet/2/40/taj-776811.pdf" H 3350 2850 50 0001 C CNN
 F 4 "AVX" H 0 0 50 0001 C CNN "MFR"
-F 5 "F931A476KAA" H 0 0 50 0001 C CNN "MPN"
-F 6 "Mouser" H 0 0 50 0001 C CNN "SPR"
-F 7 "647-F931A476KAA" H 0 0 50 0001 C CNN "SPN"
+F 5 "TAJC476K016SNJ" H 0 0 50 0001 C CNN "MPN"
+F 6 "Mouser" H 0 0 50 0001 C CNN "SPR"
+F 7 "581-TAJC476K016SNJ" H 0 0 50 0001 C CNN "SPN"
 F 8 "-" H 0 0 50 0001 C CNN "SPURL"
 	1    3350 2850
@@
 F 0 "C34" V 4675 4100 50 0000 C CNN
 F 1 "47u" V 4584 4100 50 0000 C CNN
-F 2 "Capacitors_Tantalum_SMD:CP_Tantalum_Case-A_EIA-3216-18_Reflow" H 4450 4100 50 0001 C CNN
-F 3 "https://www.mouser.de/datasheet/2/40/f93-776559.pdf" H 4450 4100 50 0001 C CNN
+F 2 "Capacitors_Tantalum_SMD:CP_EIA-6032-28_Kemet-C" H 4450 4100 50 0001 C CNN
+F 3 "https://www.mouser.de/datasheet/2/40/taj-776811.pdf" H 4450 4100 50 0001 C CNN
 F 4 "AVX" H 0 0 50 0001 C CNN "MFR"
-F 5 "F931A476KAA" H 0 0 50 0001 C CNN "MPN"
-F 6 "Mouser" H 0 0 50 0001 C CNN "SPR"
-F 7 "647-F931A476KAA" H 0 0 50 0001 C CNN "SPN"
+F 5 "TAJC476K016SNJ" H 0 0 50 0001 C CNN "MPN"
+F 6 "Mouser" H 0 0 50 0001 C CNN "SPR"
+F 7 "581-TAJC476K016SNJ" H 0 0 50 0001 C CNN "SPN"
 F 8 "-" H 0 0 50 0001 C CNN "SPURL"
 	1    4450 4100
@@
 F 0 "C36" V 4975 4100 50 0000 C CNN
 F 1 "47u" V 4884 4100 50 0000 C CNN
-F 2 "Capacitors_Tantalum_SMD:CP_Tantalum_Case-A_EIA-3216-18_Reflow" H 4750 4100 50 0001 C CNN
-F 3 "https://www.mouser.de/datasheet/2/40/f93-776559.pdf" H 4750 4100 50 0001 C CNN
+F 2 "Capacitors_Tantalum_SMD:CP_EIA-6032-28_Kemet-C" H 4750 4100 50 0001 C CNN
+F 3 "https://www.mouser.de/datasheet/2/40/taj-776811.pdf" H 4750 4100 50 0001 C CNN
 F 4 "AVX" H 0 0 50 0001 C CNN "MFR"
-F 5 "F931A476KAA" H 0 0 50 0001 C CNN "MPN"
-F 6 "Mouser" H 0 0 50 0001 C CNN "SPR"
-F 7 "647-F931A476KAA" H 0 0 50 0001 C CNN "SPN"
+F 5 "TAJC476K016SNJ" H 0 0 50 0001 C CNN "MPN"
+F 6 "Mouser" H 0 0 50 0001 C CNN "SPR"
+F 7 "581-TAJC476K016SNJ" H 0 0 50 0001 C CNN "SPN"
 F 8 "-" H 0 0 50 0001 C CNN "SPURL"
 	1    4750 4100

Commit message: Revision 0.2: Added FET for channel switching; Rename to MMDVM_RPT_Hat
Parts:
- C26, C27, C31, C34, C36: symbol MMDVM_Hat-rescue:CP_Small-device -> MMDVM_Hat-rescue:CP_Small-device-MMDVM_Hat-rescue
- C28, C29, C30, C32, C33, C35, C37, C38: symbol MMDVM_Hat-rescue:C_Small-device -> MMDVM_Hat-rescue:C_Small-device-MMDVM_Hat-rescue
- J8: symbol MMDVM_Hat-rescue:GS3-conn -> MMDVM_Hat-rescue:GS3-conn-MMDVM_Hat-rescue
- R20, R21, R22, R23, R24, R25, R26, R27, R28, R29, R30, R31, R32: symbol MMDVM_Hat-rescue:R_Small-device -> MMDVM_Hat-rescue:R_Small-device-MMDVM_Hat-rescue
- RV2, RV3, RV4: symbol MMDVM_Hat-rescue:POT-device -> MMDVM_Hat-rescue:POT-device-MMDVM_Hat-rescue
- TP2, TP3, TP4, TP5: symbol MMDVM_Hat-rescue:TEST-device -> MMDVM_Hat-rescue:TEST-device-MMDVM_Hat-rescue
- U3, U4: symbol MMDVM_Hat-rescue:MCP6002-xMS-linear -> MMDVM_Hat-rescue:MCP6002-xMS-linear-MMDVM_Hat-rescue
Changed lines of the file:
@@
 $EndDescr
 $Comp
-L MMDVM_Hat-rescue:POT-device RV2
+L MMDVM_Hat-rescue:POT-device-MMDVM_Hat-rescue RV2
 U 1 1 5BCD4E2B
 P 1150 1750
@@
 $EndComp
 $Comp
-L MMDVM_Hat-rescue:R_Small-device R21
+L MMDVM_Hat-rescue:R_Small-device-MMDVM_Hat-rescue R21
 U 1 1 5BCD4EB8
 P 1150 2100
@@
 $EndComp
 $Comp
-L MMDVM_Hat-rescue:R_Small-device R22
+L MMDVM_Hat-rescue:R_Small-device-MMDVM_Hat-rescue R22
 U 1 1 5BCD4F6A
 P 1350 1500
@@
 $EndComp
 $Comp
-L MMDVM_Hat-rescue:TEST-device TP3
+L MMDVM_Hat-rescue:TEST-device-MMDVM_Hat-rescue TP3
 U 1 1 5BCD5068
 P 1150 1400
@@
 $EndComp
 $Comp
-L MMDVM_Hat-rescue:CP_Small-device C26
+L MMDVM_Hat-rescue:CP_Small-device-MMDVM_Hat-rescue C26
 U 1 1 5BCD5130
 P 1750 1750
@@
 $EndComp
 $Comp
-L MMDVM_Hat-rescue:R_Small-device R25
+L MMDVM_Hat-rescue:R_Small-device-MMDVM_Hat-rescue R25
 U 1 1 5BCD5205
 P 1950 1550
@@
 $EndComp
 $Comp
-L MMDVM_Hat-rescue:R_Small-device R23
+L MMDVM_Hat-rescue:R_Small-device-MMDVM_Hat-rescue R23
 U 1 1 5BCD524D
 P 1700 1150
@@
 $EndComp
 $Comp
-L MMDVM_Hat-rescue:R_Small-device R24
+L MMDVM_Hat-rescue:R_Small-device-MMDVM_Hat-rescue R24
 U 1 1 5BCD5285
 P 1950 1150
@@
 $EndComp
 $Comp
-L MMDVM_Hat-rescue:CP_Small-device C27
+L MMDVM_Hat-rescue:CP_Small-device-MMDVM_Hat-rescue C27
 U 1 1 5BCD5529
 P 2250 1150
@@
 $EndComp
 $Comp
-L MMDVM_Hat-rescue:MCP6002-xMS-linear U3
+L MMDVM_Hat-rescue:MCP6002-xMS-linear-MMDVM_Hat-rescue U3
 U 2 1 5BCD6263
 P 3850 4100
@@
 $EndComp
 $Comp
-L MMDVM_Hat-rescue:MCP6002-xMS-linear U4
+L MMDVM_Hat-rescue:MCP6002-xMS-linear-MMDVM_Hat-rescue U4
 U 2 1 5BCD68DE
 P 5200 1950
@@
 $EndComp
 $Comp
-L MMDVM_Hat-rescue:POT-device RV3
+L MMDVM_Hat-rescue:POT-device-MMDVM_Hat-rescue RV3
 U 1 1 5BCD7607
 P 3350 2500
@@
 $EndComp
 $Comp
-L MMDVM_Hat-rescue:R_Small-device R29
+L MMDVM_Hat-rescue:R_Small-device-MMDVM_Hat-rescue R29
 U 1 1 5BCD7D3B
 P 3350 2100
@@
 $EndComp
 $Comp
-L MMDVM_Hat-rescue:CP_Small-device C31
+L MMDVM_Hat-rescue:CP_Small-device-MMDVM_Hat-rescue C31
 U 1 1 5BCD873A
 P 3350 2850
@@
 $EndComp
 $Comp
-L MMDVM_Hat-rescue:R_Small-device R30
+L MMDVM_Hat-rescue:R_Small-device-MMDVM_Hat-rescue R30
 U 1 1 5BCD8F1B
 P 3550 1850
@@
 $EndComp
 $Comp
-L MMDVM_Hat-rescue:C_Small-device C32
+L MMDVM_Hat-rescue:C_Small-device-MMDVM_Hat-rescue C32
 U 1 1 5BCD93D4
 P 3750 2050
@@
 $EndComp
 $Comp
-L MMDVM_Hat-rescue:R_Small-device R31
+L MMDVM_Hat-rescue:R_Small-device-MMDVM_Hat-rescue R31
 U 1 1 5BCD9D1A
 P 3950 1850
@@
 $EndComp
 $Comp
-L MMDVM_Hat-rescue:R_Small-device R32
+L MMDVM_Hat-rescue:R_Small-device-MMDVM_Hat-rescue R32
 U 1 1 5BCDA22F
 P 4350 1850
@@
 $EndComp
 $Comp
-L MMDVM_Hat-rescue:C_Small-device C33
+L MMDVM_Hat-rescue:C_Small-device-MMDVM_Hat-rescue C33
 U 1 1 5BCDCD57
 P 4150 2050
@@
 $EndComp
 $Comp
-L MMDVM_Hat-rescue:TEST-device TP4
+L MMDVM_Hat-rescue:TEST-device-MMDVM_Hat-rescue TP4
 U 1 1 5BCDE691
 P 5600 1850
@@
 $EndComp
 $Comp
-L MMDVM_Hat-rescue:C_Small-device C37
+L MMDVM_Hat-rescue:C_Small-device-MMDVM_Hat-rescue C37
 U 1 1 5BCDF28B
 P 6300 1100
@@
 $EndComp
 $Comp
-L MMDVM_Hat-rescue:C_Small-device C38
+L MMDVM_Hat-rescue:C_Small-device-MMDVM_Hat-rescue C38
 U 1 1 5BCDF324
 P 6700 1100
@@
 $EndComp
 $Comp
-L MMDVM_Hat-rescue:C_Small-device C35
+L MMDVM_Hat-rescue:C_Small-device-MMDVM_Hat-rescue C35
 U 1 1 5BCE54C1
 P 4550 2050
@@
 $EndComp
 $Comp
-L MMDVM_Hat-rescue:MCP6002-xMS-linear U3
+L MMDVM_Hat-rescue:MCP6002-xMS-linear-MMDVM_Hat-rescue U3
 U 1 1 5BCEC008
 P 1550 4000
@@
 $EndComp
 $Comp
-L MMDVM_Hat-rescue:MCP6002-xMS-linear U4
+L MMDVM_Hat-rescue:MCP6002-xMS-linear-MMDVM_Hat-rescue U4
 U 1 1 5BCEC091
 P 2950 1850
@@
 $EndComp
 $Comp
-L MMDVM_Hat-rescue:R_Small-device R20
+L MMDVM_Hat-rescue:R_Small-device-MMDVM_Hat-rescue R20
 U 1 1 5BCF132E
 P 1050 4100
@@
 $EndComp
 $Comp
-L MMDVM_Hat-rescue:TEST-device TP2
+L MMDVM_Hat-rescue:TEST-device-MMDVM_Hat-rescue TP2
 U 1 1 5BCF5161
 P 1050 3800
@@
 $EndComp
 $Comp
-L MMDVM_Hat-rescue:R_Small-device R26
+L MMDVM_Hat-rescue:R_Small-device-MMDVM_Hat-rescue R26
 U 1 1 5BCF7E46
 P 2150 4000
@@
 $EndComp
 $Comp
-L MMDVM_Hat-rescue:C_Small-device C28
+L MMDVM_Hat-rescue:C_Small-device-MMDVM_Hat-rescue C28
 U 1 1 5BCF9547
 P 2350 4200
@@
 $EndComp
 $Comp
-L MMDVM_Hat-rescue:R_Small-device R27
+L MMDVM_Hat-rescue:R_Small-device-MMDVM_Hat-rescue R27
 U 1 1 5BCFC66B
 P 2550 4000
@@
 $EndComp
 $Comp
-L MMDVM_Hat-rescue:C_Small-device C30
+L MMDVM_Hat-rescue:C_Small-device-MMDVM_Hat-rescue C30
 U 1 1 5BCFE016
 P 3150 4200
@@
 $EndComp
 $Comp
-L MMDVM_Hat-rescue:R_Small-device R28
+L MMDVM_Hat-rescue:R_Small-device-MMDVM_Hat-rescue R28
 U 1 1 5BD014BE
 P 2950 4000
@@
 $EndComp
 $Comp
-L MMDVM_Hat-rescue:C_Small-device C29
+L MMDVM_Hat-rescue:C_Small-device-MMDVM_Hat-rescue C29
 U 1 1 5BD0C5B2
 P 2750 4200
@@
 $EndComp
 $Comp
-L MMDVM_Hat-rescue:CP_Small-device C34
+L MMDVM_Hat-rescue:CP_Small-device-MMDVM_Hat-rescue C34
 U 1 1 5BD12DA5
 P 4450 4100
@@
 $EndComp
 $Comp
-L MMDVM_Hat-rescue:CP_Small-device C36
+L MMDVM_Hat-rescue:CP_Small-device-MMDVM_Hat-rescue C36
 U 1 1 5BD12ECF
 P 4750 4100
@@
 $EndComp
 $Comp
-L MMDVM_Hat-rescue:POT-device RV4
+L MMDVM_Hat-rescue:POT-device-MMDVM_Hat-rescue RV4
 U 1 1 5BD19EAC
 P 5350 4450
@@
 $EndComp
 $Comp
-L MMDVM_Hat-rescue:GS3-conn J8
+L MMDVM_Hat-rescue:GS3-conn-MMDVM_Hat-rescue J8
 U 1 1 5BD241EC
 P 5100 4100
@@
 $EndComp
 $Comp
-L MMDVM_Hat-rescue:TEST-device TP5
+L MMDVM_Hat-rescue:TEST-device-MMDVM_Hat-rescue TP5
 U 1 1 5BD2EFDA
 P 5600 3900
