File: MMDVM_RPT_Hat.sch (KiCad schematic (older format))
At the start: 73 parts, among them J1 Radio, J2 Raspberry_Pi_2_3, J3 Serial Display, J4 Panel LEDs, J5 Radio, J6 STLink, J7 GS2, Q1 IRLML2060, Q2 2N7002, Q3 IRLML2060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

Commit message: Update BOM and README for rev0.2
Parts:
- J5: MFR (none) -> Wurth Electronics; MPN (none) -> 61300811121; SPN (none) -> 710-61300811121; SPR (none) -> Mouser

Commit message: Rename CH_SW to MPOCSAG
Connections:
- net labels added: MPOCSAG
- net labels removed: CH_SW
- wire segments 353 -> 354
