File: MMDVM_RPT_Hat.kicad_pcb (KiCad board)
At the start: 2 copper layers, 65 x 56 mm, 115 parts, among them J1 Radio, J2 Raspberry_Pi_2_3, J4 Panel LEDs, J5 Radio, J7 GS2, J8 GS3, Q1 IRLML2060, Q2 2N7002, Q3 IRLML2060, U1 LD1117S33TR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

Commit message: Rename CH_SW to MPOCSAG
Parts:
- TP2: renamed from DAC TX
- TP3: renamed from Radio RX
- TP4: renamed from ADC RX
- TP5: renamed from Radio TX
- renumbered Nextion to J3, STlink to J6, TX to RV4, RSSI to TP1, TCXO to X1
Connections:
- net CH_SW renamed MPOCSAG
- J1 pad 9: Net-(J1-Pad9) -> (no net)
- J2 pad 1: Net-(J2-Pad1) -> (no net)
- J2 pad 11: Net-(J2-Pad11) -> (no net)
- J2 pad 12: Net-(J2-Pad12) -> (no net)
- J2 pad 13: Net-(J2-Pad13) -> (no net)
- J2 pad 15: Net-(J2-Pad15) -> (no net)
- J2 pad 16: Net-(J2-Pad16) -> (no net)
- J2 pad 17: Net-(J2-Pad17) -> (no net)
- J2 pad 18: Net-(J2-Pad18) -> (no net)
- J2 pad 19: Net-(J2-Pad19) -> (no net)
- J2 pad 21: Net-(J2-Pad21) -> (no net)
- J2 pad 22: Net-(J2-Pad22) -> (no net)
- J2 pad 23: Net-(J2-Pad23) -> (no net)
- J2 pad 24: Net-(J2-Pad24) -> (no net)
- J2 pad 26: Net-(J2-Pad26) -> (no net)
- J2 pad 27: Net-(J2-Pad27) -> (no net)
- J2 pad 28: Net-(J2-Pad28) -> (no net)
- J2 pad 29: Net-(J2-Pad29) -> (no net)
- J2 pad 3: Net-(J2-Pad3) -> (no net)
- J2 pad 31: Net-(J2-Pad31) -> (no net)
- J2 pad 32: Net-(J2-Pad32) -> (no net)
- J2 pad 33: Net-(J2-Pad33) -> (no net)
- J2 pad 35: Net-(J2-Pad35) -> (no net)
- J2 pad 36: Net-(J2-Pad36) -> (no net)
- J2 pad 37: Net-(J2-Pad37) -> (no net)
- J2 pad 5: Net-(J2-Pad5) -> (no net)
- J2 pad 7: Net-(J2-Pad7) -> (no net)
- U2 pad 10: Net-(U2-Pad10) -> (no net)
- U2 pad 11: Net-(U2-Pad11) -> (no net)
- U2 pad 15: Net-(U2-Pad15) -> (no net)
- U2 pad 16: Net-(U2-Pad16) -> (no net)
- U2 pad 17: Net-(U2-Pad17) -> (no net)
- U2 pad 2: Net-(U2-Pad2) -> (no net)
- U2 pad 21: Net-(U2-Pad21) -> (no net)
- U2 pad 22: Net-(U2-Pad22) -> (no net)
- U2 pad 24: Net-(U2-Pad24) -> (no net)
- U2 pad 25: Net-(U2-Pad25) -> (no net)
- U2 pad 26: Net-(U2-Pad26) -> (no net)
- U2 pad 27: Net-(U2-Pad27) -> (no net)
- U2 pad 28: Net-(U2-Pad28) -> (no net)
- U2 pad 29: Net-(U2-Pad29) -> (no net)
- U2 pad 3: Net-(U2-Pad3) -> (no net)
- U2 pad 4: Net-(U2-Pad4) -> (no net)
- U2 pad 44: Net-(U2-Pad44) -> (no net)
- U2 pad 45: Net-(U2-Pad45) -> (no net)
- U2 pad 51: Net-(U2-Pad51) -> (no net)
- U2 pad 55: Net-(U2-Pad55) -> (no net)
- U2 pad 56: Net-(U2-Pad56) -> (no net)
- U2 pad 57: Net-(U2-Pad57) -> (no net)
- U2 pad 58: Net-(U2-Pad58) -> (no net)
- U2 pad 59: Net-(U2-Pad59) -> (no net)
- U2 pad 61: Net-(U2-Pad61) -> (no net)
- U2 pad 62: Net-(U2-Pad62) -> (no net)
- U2 pad 9: Net-(U2-Pad9) -> (no net)
- X1 pad 1: Net-(X1-Pad1) -> (no net)

Commit message: Update PCB layout to rev0.3
Parts:
- added D11: FM, LEDs:LED_0603, F.Cu at (29.2, 109.6)
- added R36: 1k5, Resistors_SMD:R_0603, F.Cu at (32.8, 109.6)
- J4: footprint Pin_Headers:Pin_Header_Straight_2x10_Pitch2.00mm -> Connector_PinHeader_2.00mm:PinHeader_2x11_P2.00mm_Vertical
- moved J4 1.40 mm to (23.2, 109.0)
Connections:
- J1 pad 9: (no net) -> Net-(J1-Pad9)
- J2 pad 1: (no net) -> Net-(J2-Pad1)
- J2 pad 11: (no net) -> Net-(J2-Pad11)
- J2 pad 12: (no net) -> Net-(J2-Pad12)
- J2 pad 13: (no net) -> Net-(J2-Pad13)
- J2 pad 15: (no net) -> Net-(J2-Pad15)
- J2 pad 16: (no net) -> Net-(J2-Pad16)
- J2 pad 17: (no net) -> Net-(J2-Pad17)
- J2 pad 18: (no net) -> Net-(J2-Pad18)
- J2 pad 19: (no net) -> Net-(J2-Pad19)
- J2 pad 21: (no net) -> Net-(J2-Pad21)
- J2 pad 22: (no net) -> Net-(J2-Pad22)
- J2 pad 23: (no net) -> Net-(J2-Pad23)
- J2 pad 24: (no net) -> Net-(J2-Pad24)
- J2 pad 26: (no net) -> Net-(J2-Pad26)
- J2 pad 27: (no net) -> Net-(J2-Pad27)
- J2 pad 28: (no net) -> Net-(J2-Pad28)
- J2 pad 29: (no net) -> Net-(J2-Pad29)
- J2 pad 3: (no net) -> Net-(J2-Pad3)
- J2 pad 31: (no net) -> Net-(J2-Pad31)
- J2 pad 32: (no net) -> Net-(J2-Pad32)
- J2 pad 33: (no net) -> Net-(J2-Pad33)
- J2 pad 35: (no net) -> Net-(J2-Pad35)
- J2 pad 36: (no net) -> Net-(J2-Pad36)
- J2 pad 37: (no net) -> Net-(J2-Pad37)
- J2 pad 5: (no net) -> Net-(J2-Pad5)
- J2 pad 7: (no net) -> Net-(J2-Pad7)
- J4 pad 1: Net-(D10-Pad2) -> Net-(D11-Pad2)
- J4 pad 11: Net-(D9-Pad2) -> Net-(D8-Pad2)
- J4 pad 13: Net-(D4-Pad2) -> Net-(D9-Pad2)
- J4 pad 15: Net-(D3-Pad2) -> Net-(D4-Pad2)
- J4 pad 17: Net-(D2-Pad2) -> Net-(D3-Pad2)
- J4 pad 19: Net-(D1-Pad2) -> Net-(D2-Pad2)
- J4 pad 3: Net-(D5-Pad2) -> Net-(D10-Pad2)
- J4 pad 5: Net-(D6-Pad2) -> Net-(D5-Pad2)
- J4 pad 7: Net-(D7-Pad2) -> Net-(D6-Pad2)
- J4 pad 9: Net-(D8-Pad2) -> Net-(D7-Pad2)
- U2 pad 10: (no net) -> Net-(U2-Pad10)
- U2 pad 11: (no net) -> Net-(U2-Pad11)
- U2 pad 15: (no net) -> Net-(U2-Pad15)
- U2 pad 16: (no net) -> Net-(U2-Pad16)
- U2 pad 17: (no net) -> Net-(U2-Pad17)
- U2 pad 2: (no net) -> Net-(U2-Pad2)
- U2 pad 21: (no net) -> Net-(U2-Pad21)
- U2 pad 22: (no net) -> Net-(U2-Pad22)
- U2 pad 24: (no net) -> Net-(U2-Pad24)
- U2 pad 25: (no net) -> Net-(U2-Pad25)
- U2 pad 26: (no net) -> Net-(U2-Pad26)
- U2 pad 27: (no net) -> Net-(U2-Pad27)
- U2 pad 28: (no net) -> Net-(U2-Pad28)
- U2 pad 29: (no net) -> Net-(U2-Pad29)
- U2 pad 3: (no net) -> Net-(U2-Pad3)
- U2 pad 4: (no net) -> Net-(U2-Pad4)
- U2 pad 44: (no net) -> FM_LED
- U2 pad 45: (no net) -> Net-(U2-Pad45)
- U2 pad 51: (no net) -> Net-(U2-Pad51)
- U2 pad 55: (no net) -> Net-(U2-Pad55)
- U2 pad 56: (no net) -> Net-(U2-Pad56)
- U2 pad 57: (no net) -> Net-(U2-Pad57)
- U2 pad 58: (no net) -> Net-(U2-Pad58)
- U2 pad 59: (no net) -> Net-(U2-Pad59)
- U2 pad 61: (no net) -> Net-(U2-Pad61)
- U2 pad 62: (no net) -> Net-(U2-Pad62)
- U2 pad 9: (no net) -> Net-(U2-Pad9)
- X1 pad 1: (no net) -> Net-(X1-Pad1)
Routing:
- net FM_LED: track 0.00 -> 20.1 mm
- net Net-(D11-Pad2): track 0.00 -> 10.2 mm, vias 0 -> 1
- net PTT: track 50.5 -> 47.6 mm
- net SWDIO: track 43.5 -> 42.6 mm
- net GND: vias 62 -> 64
Other:
- board text added: "FM"
- board text added: "Revision 0.3"
- board text removed: "Revision 0.2"

Commit message: Re-add OSHW and KiCad logos as well as drill file
Parts:
- added REF**: KiCad-Logo2_8mm_SilkScreen, Symbol:KiCad-Logo2_8mm_SilkScreen, B.Cu at (74.0, 101.6)
- added REF**: OSHW-Logo_28.5x30mm_SilkScreen, Symbol:OSHW-Logo_28.5x30mm_SilkScreen, B.Cu at (49.8, 92.2)
